File: KiCAD/Capacitors.kicad_sch (KiCad schematic)
At the start: 48 parts

Commit message: Update to V9
Parts:
- renumbered Z9 to Z52, Z44 to Z72, Z60 to Z72
Connections:
- net GND: now also Z24.4, Z24.5; no longer Z24.12, Z24.13
Changed lines of the file:
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@@
 (kicad_sch
-	(version 20231120)
+	(version 20250114)
 	(generator "eeschema")
-	(generator_version "8.0")
+	(generator_version "9.0")
 	(paper "USLetter")
 	(title_block
@@
 		(on_board yes)
 		(dnp no)
-		(property "Reference" "Z9"
+		(property "Reference" "Z52"
 			(at 53.975 164.465 0)
 			(effects
@@
 		(lib_id "74xx:74LS132")
 		(at 31.115 156.21 0)
-		(unit 4)
+		(unit 2)
 		(exclude_from_sim no)
 		(in_bom yes)
@@
 		(on_board yes)
 		(dnp no)
-		(property "Reference" "Z44"
+		(property "Reference" "Z72"
 			(at 54.102 174.752 0)
 			(effects
@@
 		(dnp no)
 		(fields_autoplaced yes)
-		(property "Reference" "#PWR01"
+		(property "Reference" "#PWR042"
 			(at 22.225 110.49 0)
 			(effects
@@
 		(on_board yes)
 		(dnp no)
-		(property "Reference" "Z60"
+		(property "Reference" "Z72"
 			(at 140.97 33.655 0)
 			(effects
@@
 		(on_board yes)
 		(dnp no)
-		(property "Reference" "#PWR01"
+		(property "Reference" "#PWR045"
 			(at 22.225 140.97 0)
 			(effects
