File: KiCAD/Power.kicad_sch (KiCad schematic)
At the start: 41 parts, among them J1 Front View, Q3 TIP29A, Q4 2N6594, Q5 2N3906, Q6 MJE34

Commit message: Update to V9
Changed lines of the file:
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@@
 (kicad_sch
-	(version 20231120)
+	(version 20250114)
 	(generator "eeschema")
-	(generator_version "8.0")
+	(generator_version "9.0")
 	(paper "USLetter")
 	(title_block
@@
 		(comment 4 "Power")
 	)
+	(text "12V-20V AC\n1A"
+		(exclude_from_sim no)
+		(at 51.435 81.28 0)
+		(effects
+			(font
+				(size 1 1)
+			)
+			(justify right bottom)
+		)
+	)
+	(text "2W"
+		(exclude_from_sim no)
+		(at 216.535 103.505 0)
+		(effects
+			(font
+				(size 1 1)
+			)
+			(justify left bottom)
+		)
+	)
+	(text "0.5W"
+		(exclude_from_sim no)
+		(at 105.41 185.42 0)
+		(effects
+			(font
+				(size 1 1)
+			)
+			(justify left bottom)
+		)
+	)
+	(text "3W"
+		(exclude_from_sim no)
+		(at 207.01 26.035 0)
+		(effects
+			(font
+				(size 1 1)
+			)
+			(justify left bottom)
+		)
+	)
+	(text "0.5W"
+		(exclude_from_sim no)
+		(at 182.245 112.395 0)
+		(effects
+			(font
+				(size 1 1)
+			)
+			(justify left bottom)
+		)
+	)
+	(text "14V-20V DC\n350mA"
+		(exclude_from_sim no)
+		(at 34.29 93.98 0)
+		(effects
+			(font
+				(size 1 1)
+			)
+			(justify left bottom)
+		)
+	)
 	(junction
 		(at 165.735 165.1)
@@
 		)
 	)
-	(text "12V-20V AC\n1A"
-		(exclude_from_sim no)
-		(at 51.435 81.28 0)
-		(effects
-			(font
-				(size 1 1)
-			)
-			(justify right bottom)
-		)
-	)
-	(text "2W"
-		(exclude_from_sim no)
-		(at 216.535 103.505 0)
-		(effects
-			(font
-				(size 1 1)
-			)
-			(justify left bottom)
-		)
-	)
-	(text "0.5W"
-		(exclude_from_sim no)
-		(at 105.41 185.42 0)
-		(effects
-			(font
-				(size 1 1)
-			)
-			(justify left bottom)
-		)
-	)
-	(text "3W"
-		(exclude_from_sim no)
-		(at 207.01 26.035 0)
-		(effects
-			(font
-				(size 1 1)
-			)
-			(justify left bottom)
-		)
-	)
-	(text "0.5W"
-		(exclude_from_sim no)
-		(at 182.245 112.395 0)
-		(effects
-			(font
-				(size 1 1)
-			)
-			(justify left bottom)
-		)
-	)
-	(text "14V-20V DC\n350mA"
-		(exclude_from_sim no)
-		(at 34.29 93.98 0)
-		(effects
-			(font
-				(size 1 1)
-			)
-			(justify left bottom)
-		)
-	)
 	(symbol
 		(lib_id "Device:R_Potentiometer")
@@
 		(dnp no)
 		(fields_autoplaced yes)
-		(property "Reference" "#FLG01"
+		(property "Reference" "#FLG06"
 			(at 178.435 32.385 0)
 			(effects
@@
 		(dnp no)
 		(fields_autoplaced yes)
-		(property "Reference" "#FLG01"
+		(property "Reference" "#FLG04"
 			(at 247.015 135.89 0)
 			(effects
@@
 		(on_board yes)
 		(dnp no)
-		(property "Reference" "#PWR01"
+		(property "Reference" "#PWR0187"
 			(at 151.13 172.085 0)
 			(effects
@@
 		(dnp no)
 		(fields_autoplaced yes)
-		(property "Reference" "#PWR01"
+		(property "Reference" "#PWR0185"
 			(at 99.695 202.565 0)
 			(effects
@@
 		(dnp no)
 		(fields_autoplaced yes)
-		(property "Reference" "#FLG01"
+		(property "Reference" "#FLG07"
 			(at 86.995 20.955 0)
 			(effects
@@
 		(dnp no)
 		(fields_autoplaced yes)
-		(property "Reference" "#FLG01"
+		(property "Reference" "#FLG03"
 			(at 241.3 20.955 0)
 			(effects
@@
 		(dnp no)
 		(fields_autoplaced yes)
-		(property "Reference" "#PWR01"
+		(property "Reference" "#PWR0184"
 			(at 55.245 90.551 0)
 			(effects
@@
 		(on_board yes)
 		(dnp no)
-		(property "Reference" "#PWR01"
+		(property "Reference" "#PWR0190"
 			(at 151.13 81.28 0)
 			(effects
@@
 		(dnp no)
 		(fields_autoplaced yes)
-		(property "Reference" "#FLG01"
+		(property "Reference" "#FLG05"
 			(at 142.875 180.34 0)
 			(effects
@@
 		(dnp no)
 		(fields_autoplaced yes)
-		(property "Reference" "#FLG01"
+		(property "Reference" "#FLG08"
 			(at 151.13 98.425 0)
 			(effects
