File: KiCAD/VideoSync.kicad_sch (KiCad schematic)
At the start: 11 parts

Commit message: Update to V9
Changed lines of the file:
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@@
 (kicad_sch
-	(version 20231120)
+	(version 20250114)
 	(generator "eeschema")
-	(generator_version "8.0")
+	(generator_version "9.0")
 	(paper "USLetter")
 	(title_block
@@
 		(comment 4 "Video Sync")
 	)
+	(rectangle
+		(start 158.115 48.895)
+		(end 171.45 126.365)
+		(stroke
+			(width 0)
+			(type dot)
+		)
+		(fill
+			(type none)
+		)
+	)
+	(rectangle
+		(start 100.33 55.245)
+		(end 149.225 120.015)
+		(stroke
+			(width 0)
+			(type dot)
+		)
+		(fill
+			(type none)
+		)
+	)
+	(rectangle
+		(start 53.34 71.755)
+		(end 93.345 102.87)
+		(stroke
+			(width 0)
+			(type dot)
+		)
+		(fill
+			(type none)
+		)
+	)
+	(rectangle
+		(start 175.895 60.96)
+		(end 254 113.665)
+		(stroke
+			(width 0)
+			(type dot)
+		)
+		(fill
+			(type none)
+		)
+	)
+	(text "Amplifier"
+		(exclude_from_sim no)
+		(at 53.975 71.12 0)
+		(effects
+			(font
+				(size 1 1)
+			)
+			(justify left bottom)
+		)
+	)
+	(text "Sync Offset"
+		(exclude_from_sim no)
+		(at 100.965 54.61 0)
+		(effects
+			(font
+				(size 1 1)
+			)
+			(justify left bottom)
+		)
+	)
+	(text "H-Sync"
+		(exclude_from_sim no)
+		(at 189.865 76.835 0)
+		(effects
+			(font
+				(size 1 1)
+			)
+			(justify left bottom)
+		)
+	)
+	(text "V-Sync\nOffset\nCapacitor"
+		(exclude_from_sim no)
+		(at 130.175 116.84 0)
+		(effects
+			(font
+				(size 1 1)
+			)
+			(justify left bottom)
+		)
+	)
+	(text "V-Sync"
+		(exclude_from_sim no)
+		(at 190.5 98.425 0)
+		(effects
+			(font
+				(size 1 1)
+			)
+			(justify left bottom)
+		)
+	)
+	(text "Inv-Sync"
+		(exclude_from_sim no)
+		(at 201.93 87.63 0)
+		(effects
+			(font
+				(size 1 1)
+			)
+			(justify left bottom)
+		)
+	)
+	(text "H-Sync\nOffset\nCapacitor"
+		(exclude_from_sim no)
+		(at 130.175 62.865 0)
+		(effects
+			(font
+				(size 1 1)
+			)
+			(justify left bottom)
+		)
+	)
+	(text "Sync Pulse Length"
+		(exclude_from_sim no)
+		(at 158.115 48.26 0)
+		(effects
+			(font
+				(size 1 1)
+			)
+			(justify left bottom)
+		)
+	)
+	(text "V-Sync\nLength"
+		(exclude_from_sim no)
+		(at 159.385 104.14 0)
+		(effects
+			(font
+				(size 1 1)
+			)
+			(justify left bottom)
+		)
+	)
+	(text "V-Sync Offset\nResistor"
+		(exclude_from_sim no)
+		(at 101.6 92.71 0)
+		(effects
+			(font
+				(size 1 1)
+			)
+			(justify left bottom)
+		)
+	)
+	(text "H-Sync\nLength"
+		(exclude_from_sim no)
+		(at 159.385 74.295 0)
+		(effects
+			(font
+				(size 1 1)
+			)
+			(justify left bottom)
+		)
+	)
+	(text "Combine Sync Signals"
+		(exclude_from_sim no)
+		(at 176.53 60.325 0)
+		(effects
+			(font
+				(size 1 1)
+			)
+			(justify left bottom)
+		)
+	)
+	(text "H-Sync Offset\nResistor"
+		(exclude_from_sim no)
+		(at 102.235 74.803 0)
+		(effects
+			(font
+				(size 1 1)
+			)
+			(justify left bottom)
+		)
+	)
 	(junction
 		(at 114.935 107.315)
@@
 		)
 	)
-	(rectangle
-		(start 158.115 48.895)
-		(end 171.45 126.365)
-		(stroke
-			(width 0)
-			(type dot)
-		)
-		(fill
-			(type none)
-		)
-	)
-	(rectangle
-		(start 100.33 55.245)
-		(end 149.225 120.015)
-		(stroke
-			(width 0)
-			(type dot)
-		)
-		(fill
-			(type none)
-		)
-	)
-	(rectangle
-		(start 53.34 71.755)
-		(end 93.345 102.87)
-		(stroke
-			(width 0)
-			(type dot)
-		)
-		(fill
-			(type none)
-		)
-	)
-	(rectangle
-		(start 175.895 60.96)
-		(end 254 113.665)
-		(stroke
-			(width 0)
-			(type dot)
-		)
-		(fill
-			(type none)
-		)
-	)
-	(text "Amplifier"
-		(exclude_from_sim no)
-		(at 53.975 71.12 0)
-		(effects
-			(font
-				(size 1 1)
-			)
-			(justify left bottom)
-		)
-	)
-	(text "Sync Offset"
-		(exclude_from_sim no)
-		(at 100.965 54.61 0)
-		(effects
-			(font
-				(size 1 1)
-			)
-			(justify left bottom)
-		)
-	)
-	(text "H-Sync"
-		(exclude_from_sim no)
-		(at 189.865 76.835 0)
-		(effects
-			(font
-				(size 1 1)
-			)
-			(justify left bottom)
-		)
-	)
-	(text "V-Sync\nOffset\nCapacitor"
-		(exclude_from_sim no)
-		(at 130.175 116.84 0)
-		(effects
-			(font
-				(size 1 1)
-			)
-			(justify left bottom)
-		)
-	)
-	(text "V-Sync"
-		(exclude_from_sim no)
-		(at 190.5 98.425 0)
-		(effects
-			(font
-				(size 1 1)
-			)
-			(justify left bottom)
-		)
-	)
-	(text "Inv-Sync"
-		(exclude_from_sim no)
-		(at 201.93 87.63 0)
-		(effects
-			(font
-				(size 1 1)
-			)
-			(justify left bottom)
-		)
-	)
-	(text "H-Sync\nOffset\nCapacitor"
-		(exclude_from_sim no)
-		(at 130.175 62.865 0)
-		(effects
-			(font
-				(size 1 1)
-			)
-			(justify left bottom)
-		)
-	)
-	(text "Sync Pulse Length"
-		(exclude_from_sim no)
-		(at 158.115 48.26 0)
-		(effects
-			(font
-				(size 1 1)
-			)
-			(justify left bottom)
-		)
-	)
-	(text "V-Sync\nLength"
-		(exclude_from_sim no)
-		(at 159.385 104.14 0)
-		(effects
-			(font
-				(size 1 1)
-			)
-			(justify left bottom)
-		)
-	)
-	(text "V-Sync Offset\nResistor"
-		(exclude_from_sim no)
-		(at 101.6 92.71 0)
-		(effects
-			(font
-				(size 1 1)
-			)
-			(justify left bottom)
-		)
-	)
-	(text "H-Sync\nLength"
-		(exclude_from_sim no)
-		(at 159.385 74.295 0)
-		(effects
-			(font
-				(size 1 1)
-			)
-			(justify left bottom)
-		)
-	)
-	(text "Combine Sync Signals"
-		(exclude_from_sim no)
-		(at 176.53 60.325 0)
-		(effects
-			(font
-				(size 1 1)
-			)
-			(justify left bottom)
-		)
-	)
-	(text "H-Sync Offset\nResistor"
-		(exclude_from_sim no)
-		(at 102.235 74.803 0)
-		(effects
-			(font
-				(size 1 1)
-			)
-			(justify left bottom)
-		)
-	)
 	(hierarchical_label "VDRV"
 		(shape input)
 		(at 60.96 95.885 180)
-		(fields_autoplaced yes)
 		(effects
 			(font
@@
 		(shape input)
 		(at 60.96 79.375 180)
-		(fields_autoplaced yes)
 		(effects
 			(font
@@
 		(shape output)
 		(at 245.745 87.63 0)
-		(fields_autoplaced yes)
 		(effects
 			(font
@@
 		(on_board yes)
 		(dnp no)
-		(property "Reference" "#PWR04"
+		(property "Reference" "#PWR0140"
 			(at 168.275 126.365 0)
 			(effects
@@
 		(on_board yes)
 		(dnp no)
-		(property "Reference" "#PWR03"
+		(property "Reference" "#PWR0139"
 			(at 168.275 48.895 0)
 			(effects
